Commit message: update urdf&xml

File: urdf/atom02.urdf (robot description, URDF)
Before this commit: robot ATOM02, 25 links, 24 joints
Links:
- removed link left_elbow_pitch_link
- removed link left_elbow_yaw_link
- removed link left_thigh_pitch_link
- removed link left_thigh_roll_link
- removed link left_thigh_yaw_link
- removed link right_elbow_pitch_link
- removed link right_elbow_yaw_link
- removed link right_thigh_pitch_link
- removed link right_thigh_roll_link
- removed link right_thigh_yaw_link
- removed link torso_roll_link
- removed link torso_yaw_link
- added link left_elbow_link, mass 0.73978; collision mesh filename=../meshes/left_elbow_link_collision.stl; visual mesh filename=../meshes/left_elbow_link_visual.stl
- added link left_hip_pitch_link, mass 1.45119; collision mesh filename=../meshes/left_hip_pitch_link_collision.stl; visual mesh filename=../meshes/left_hip_pitch_link_visual.stl
- added link left_hip_roll_link, mass 1.9198; collision mesh filename=../meshes/left_hip_roll_link_collision.stl; visual mesh filename=../meshes/left_hip_roll_link_visual.stl
- added link left_hip_yaw_link, mass 2.33885; collision mesh filename=../meshes/left_hip_yaw_link_collision.stl; visual mesh filename=../meshes/left_hip_yaw_link_visual.stl
- added link left_wrist_link, mass 0.2189; collision mesh filename=../meshes/left_wrist_link_collision.stl; visual mesh filename=../meshes/left_wrist_link_visual.stl
- added link right_elbow_link, mass 0.739789; collision mesh filename=../meshes/right_elbow_link_collision.stl; visual mesh filename=../meshes/right_elbow_link_visual.stl
- added link right_hip_pitch_link, mass 1.45119; collision mesh filename=../meshes/right_hip_pitch_link_collision.stl; visual mesh filename=../meshes/right_hip_pitch_link_visual.stl
- added link right_hip_roll_link, mass 1.92071; collision mesh filename=../meshes/right_hip_roll_link_collision.stl; visual mesh filename=../meshes/right_hip_roll_link_visual.stl
- added link right_hip_yaw_link, mass 2.33884; collision mesh filename=../meshes/right_hip_yaw_link_collision.stl; visual mesh filename=../meshes/right_hip_yaw_link_visual.stl
- added link right_wrist_link, mass 0.2189; collision mesh filename=../meshes/right_wrist_link_collision.stl; visual mesh filename=../meshes/right_wrist_link_visual.stl
- added link waist_roll_link, mass 1.48989; collision mesh filename=../meshes/waist_roll_link_collision.stl; visual mesh filename=../meshes/waist_roll_link_visual.stl
- added link waist_yaw_link, mass 6.09562; collision mesh filename=../meshes/waist_yaw_link_collision.stl; visual mesh filename=../meshes/waist_yaw_link_visual.stl
- link base_link: mass 3.23595958 -> 3.2691; geometry collision mesh filename=../meshes/base_link_collision.stl; visual mesh filename=../meshes/base_link_visual.stl
- link left_ankle_pitch_link: mass 0.22519575 -> 0.169597; geometry collision mesh filename=../meshes/left_ankle_pitch_link_collision.stl; visual mesh filename=../meshes/left_ankle_pitch_link_visual.stl
- link left_ankle_roll_link: mass 0.58290878 -> 0.582932; geometry collision mesh filename=../meshes/left_ankle_roll_link_collision.stl; visual mesh filename=../meshes/left_ankle_roll_link_visual.stl
- link left_knee_link: mass 2.18421456 -> 2.25436; geometry collision mesh filename=../meshes/left_knee_link_collision.stl; visual mesh filename=../meshes/left_knee_link_visual.stl
- link left_shoulder_pitch_link: mass 0.68492195 -> 0.669577; geometry collision mesh filename=../meshes/left_shoulder_pitch_link_collision.stl; visual mesh filename=../meshes/left_shoulder_pitch_link_visual.stl
- link left_shoulder_roll_link: mass 0.69553781 -> 0.678239; geometry collision mesh filename=../meshes/left_shoulder_roll_link_collision.stl; visual mesh filename=../meshes/left_shoulder_roll_link_visual.stl
- link left_shoulder_yaw_link: mass 1.01870173 -> 0.905342; geometry collision mesh filename=../meshes/left_shoulder_yaw_link_collision.stl; visual mesh filename=../meshes/left_shoulder_yaw_link_visual.stl
- link right_ankle_pitch_link: mass 0.22519575 -> 0.169597; geometry collision mesh filename=../meshes/right_ankle_pitch_link_collision.stl; visual mesh filename=../meshes/right_ankle_pitch_link_visual.stl
- link right_ankle_roll_link: mass 0.58290878 -> 0.607702; geometry collision mesh filename=../meshes/right_ankle_roll_link_collision.stl; visual mesh filename=../meshes/right_ankle_roll_link_visual.stl
- link right_knee_link: mass 2.16342478 -> 2.24966; geometry collision mesh filename=../meshes/right_knee_link_collision.stl; visual mesh filename=../meshes/right_knee_link_visual.stl
- link right_shoulder_pitch_link: mass 0.68494995 -> 0.669577; geometry collision mesh filename=../meshes/right_shoulder_pitch_link_collision.stl; visual mesh filename=../meshes/right_shoulder_pitch_link_visual.stl
- link right_shoulder_roll_link: mass 0.70646494 -> 0.678176; geometry collision mesh filename=../meshes/right_shoulder_roll_link_collision.stl; visual mesh filename=../meshes/right_shoulder_roll_link_visual.stl
- link right_shoulder_yaw_link: mass 1.02101321 -> 0.905341; geometry collision mesh filename=../meshes/right_shoulder_yaw_link_collision.stl; visual mesh filename=../meshes/right_shoulder_yaw_link_visual.stl
Joints:
- removed joint left_elbow_pitch_joint
- removed joint left_elbow_yaw_joint
- removed joint left_thigh_pitch_joint
- removed joint left_thigh_roll_joint
- removed joint left_thigh_yaw_joint
- removed joint right_elbow_pitch_joint
- removed joint right_elbow_yaw_joint
- removed joint right_thigh_pitch_joint
- removed joint right_thigh_roll_joint
- removed joint right_thigh_yaw_joint
- removed joint torso_roll_joint
- removed joint torso_yaw_joint
- added joint left_elbow_joint: type revolute, parent left_shoulder_yaw_link, child left_elbow_link, origin xyz=0.00943981 -0.027125 0.126934 rpy=1.5708 3.45984e-15 4.67243e-13, axis 0 0 1, limit lower=-1 upper=3.14 effort=10 velocity=10
- added joint left_hip_pitch_joint: type revolute, parent base_link, child left_hip_pitch_link, origin xyz=0.0439249 0.0712663 -0.0347123 rpy=-1.5708 -3.15315e-15 -2.24154e-15, axis 0 0 1, limit lower=-2.862 upper=2.862 effort=10 velocity=10
- added joint left_hip_roll_joint: type revolute, parent left_hip_pitch_link, child left_hip_roll_link, origin xyz=0.0327788 4.92661e-16 0.057104 rpy=-1.5708 1.20684e-16 -1.5708, axis 0 0 1, limit lower=-0.1745 upper=2.6878 effort=10 velocity=10
- added joint left_hip_yaw_joint: type revolute, parent left_hip_roll_link, child left_hip_yaw_link, origin xyz=-0.137165 2.62981e-11 -0.0125459 rpy=2.31122e-13 -1.5708 0, axis 0 0 1, limit lower=-1.9199 upper=1.9199 effort=10 velocity=10
- added joint left_wrist_joint: type revolute, parent left_elbow_link, child left_wrist_link, origin xyz=0.105925 0.0128812 -0.027201 rpy=-1.5708 -2.57662e-10 -1.5708, axis 0 0 1, limit lower=-3.14 upper=3.14 effort=10 velocity=10
- added joint right_elbow_joint: type revolute, parent right_shoulder_yaw_link, child right_elbow_link, origin xyz=0.00943951 0.027125 0.126934 rpy=-1.5708 -8.4185e-14 -7.15129e-13, axis 0 0 1, limit lower=-3.14 upper=1 effort=10 velocity=10
- added joint right_hip_pitch_joint: type revolute, parent base_link, child right_hip_pitch_link, origin xyz=0.0439249 -0.0687337 -0.0347123 rpy=1.5708 2.9976e-15 -7.25858e-16, axis 0 0 1, limit lower=-2.862 upper=2.862 effort=10 velocity=10
- added joint right_hip_roll_joint: type revolute, parent right_hip_pitch_link, child right_hip_roll_link, origin xyz=0.0327788 4.54498e-15 0.057104 rpy=1.5708 -1.0948e-14 1.5708, axis 0 0 1, limit lower=-2.6878 upper=0.1745 effort=10 velocity=10
- added joint right_hip_yaw_joint: type revolute, parent right_hip_roll_link, child right_hip_yaw_link, origin xyz=-0.137165 3.82238e-10 -0.0125459 rpy=-1.15743e-15 -1.5708 0, axis 0 0 1, limit lower=-1.9199 upper=1.9199 effort=10 velocity=10
- added joint right_wrist_joint: type revolute, parent right_elbow_link, child right_wrist_link, origin xyz=0.105895 -0.0134505 -0.027201 rpy=1.5708 6.44005e-14 1.5708, axis 0 0 1, limit lower=-3.14 upper=3.14 effort=10 velocity=10
- added joint waist_roll_joint: type revolute, parent base_link, child waist_roll_link, origin xyz=0.0745499 0.00126629 0.0602877 rpy=3.14159 -1.5708 0, axis 0 0 1, limit lower=-0.7854 upper=0.7854 effort=10 velocity=10
- added joint waist_yaw_joint: type revolute, parent waist_roll_link, child waist_yaw_link, origin xyz=0.0555 3.49805e-10 -0.0309136 rpy=1.25439e-13 -1.5708 0, axis 0 0 1, limit lower=-3.14 upper=3.14 effort=10 velocity=10
- joint left_ankle_pitch_joint: axis 0 -1 0 -> 0 0 1; limit lower=-0.5236 upper=0.6981 effort=60 velocity=12 -> lower=-0.6981 upper=0.5236 effort=10 velocity=10; origin xyz=0.00538908374941682 0 -0.310500012478865 rpy=0 0 0 -> xyz=-0.00142753 -0.310543 -0.03575 rpy=3.14159 -2.95771e-13 -0.0219512
- joint left_ankle_roll_joint: axis 1 0 0 -> 0 0 1; limit lower=-0.2618 upper=0.2618 effort=60 velocity=12 -> lower=-0.2618 upper=0.2618 effort=10 velocity=10; origin xyz=0.000288640584767348 0 -0.018968626966601 rpy=0 0 0 -> xyz=-0.0005 0.0189686 0 rpy=-1.5708 -9.17325e-15 -1.5708
- joint left_knee_joint: axis 0 -1 0 -> 0 0 1; limit lower=-2.7925 upper=0.2618 effort=140 velocity=12 -> lower=-2.7925 upper=0.2618 effort=10 velocity=10; origin xyz=-0.0259105994324788 0 -0.315911806813306 rpy=0 0 0 -> xyz=-0.0259106 0.0357744 0.178747 rpy=-1.5708 0.0219512 -1.19101e-15; parent left_thigh_yaw_link -> left_hip_yaw_link
- joint left_shoulder_pitch_joint: axis 0 0.999048221581858 0.0436193873653277 -> 0 0 1; limit lower=-2.9671 upper=2.6180 effort=30 velocity=12 -> lower=-3.14 upper=3.14 effort=10 velocity=10; origin xyz=-0.00531236834996837 0 0.257475047221614 rpy=0 0 0 -> xyz=-0.005 -0.101374 -0.210901 rpy=1.61443 8.09062e-06 3.52937e-07; parent torso_yaw_link -> waist_yaw_link
- joint left_shoulder_roll_joint: axis 1 0 0 -> 0 0 1; limit lower=-0.1745 upper=3.14159 effort=30 velocity=12 -> lower=-0.1745 upper=3.14 effort=10 velocity=10; origin xyz=0 0.157727108635355 0.0064438018083768 rpy=0 0 0 -> xyz=0.0272216 -4.59632e-14 0.0607 rpy=-1.5708 -9.6978e-14 -1.5708
- joint left_shoulder_yaw_joint: axis 0 0 -1 -> 0 0 1; limit lower=-3.14159 upper=3.14159 effort=30 velocity=12 -> lower=-3.14 upper=3.14 effort=10 velocity=10; origin xyz=0 0.00647177026748297 0.000725276071402214 rpy=0 0 0 -> xyz=-0.10319 -0.00197277 -0.0276539 rpy=0.000321084 -1.57079 -0.0439493
- joint right_ankle_pitch_joint: axis 0 1 0 -> 0 0 1; limit lower=-0.6981 upper=0.5236 effort=60 velocity=12 -> lower=-0.6981 upper=0.5236 effort=10 velocity=10; origin xyz=0.00538908374941711 0 -0.310500012478865 rpy=0 0 0 -> xyz=0.0122031 0.310307 -0.03575 rpy=-4.6833e-08 5.58011e-15 -0.0219512
- joint right_ankle_roll_joint: axis 1 0 0 -> 0 0 1; limit lower=-0.2618 upper=0.2618 effort=60 velocity=12 -> lower=-0.2618 upper=0.2618 effort=10 velocity=10; origin xyz=0.000288640584765455 0 -0.0189686150614563 rpy=0 0 0 -> xyz=-0.0005 0.0189686 2.77556e-17 rpy=-1.5708 5.155e-16 -1.5708
- joint right_knee_joint: axis 0 1 0 -> 0 0 1; limit lower=-0.2618 upper=2.7925 effort=140 velocity=12 -> lower=-0.2618 upper=2.7925 effort=10 velocity=10; origin xyz=-0.0259105994325459 0 -0.315911818718635 rpy=0 0 0 -> xyz=-0.0259106 -0.0357744 0.178747 rpy=1.5708 -0.0219512 2.2676e-07; parent right_thigh_yaw_link -> right_hip_yaw_link
- joint right_shoulder_pitch_joint: axis 0 -0.999048221581858 0.0436193873653299 -> 0 0 1; limit lower=-2.6180 upper=2.9671 effort=30 velocity=12 -> lower=-3.14 upper=3.14 effort=10 velocity=10; origin xyz=-0.00531236834996837 0 0.257475047221614 rpy=0 0 0 -> xyz=-0.00499971 0.101374 -0.210901 rpy=-1.61443 -8.09062e-06 3.52937e-07; parent torso_yaw_link -> waist_yaw_link
- joint right_shoulder_roll_joint: axis 1 0 0 -> 0 0 1; limit lower=-3.14159 upper=0.1745 effort=30 velocity=12 -> lower=-3.14 upper=0.1745 effort=10 velocity=10; origin xyz=0 -0.157731572169751 0.00634362168986959 rpy=0 0 0 -> xyz=0.0267216 -3.47219e-10 0.0607 rpy=1.5708 -5.91957e-14 1.5708
- joint right_shoulder_yaw_joint: axis 0 0 -1 -> 0 0 1; limit lower=-3.14159 upper=3.14159 effort=30 velocity=12 -> lower=-3.14 upper=3.14 effort=10 velocity=10; origin xyz=0 -0.00647168056291525 0.000825647150946768 rpy=0 0 0 -> xyz=-0.10319 0.0019726 -0.0276537 rpy=0.00608941 -1.57079 0.0375388

Commit message: update effort&velocity limits

File: urdf/atom02.urdf (robot description, URDF)
Before this commit: robot atom02, 25 links, 24 joints
Joints:
- joint left_ankle_pitch_joint: limit lower=-0.6981 upper=0.5236 effort=10 velocity=10 -> lower=-0.6981 upper=0.5236 effort=30 velocity=12
- joint left_ankle_roll_joint: limit lower=-0.2618 upper=0.2618 effort=10 velocity=10 -> lower=-0.2618 upper=0.2618 effort=30 velocity=12
- joint left_elbow_joint: limit lower=-1 upper=3.14 effort=10 velocity=10 -> lower=-1 upper=3.14 effort=30 velocity=12
- joint left_hip_pitch_joint: limit lower=-2.862 upper=2.862 effort=10 velocity=10 -> lower=-2.862 upper=2.862 effort=120 velocity=25
- joint left_hip_roll_joint: limit lower=-0.1745 upper=2.6878 effort=10 velocity=10 -> lower=-0.1745 upper=2.6878 effort=120 velocity=25
- joint left_hip_yaw_joint: limit lower=-1.9199 upper=1.9199 effort=10 velocity=10 -> lower=-1.9199 upper=1.9199 effort=120 velocity=25
- joint left_knee_joint: limit lower=-2.7925 upper=0.2618 effort=10 velocity=10 -> lower=-2.7925 upper=0.2618 effort=120 velocity=25
- joint left_shoulder_pitch_joint: limit lower=-3.14 upper=3.14 effort=10 velocity=10 -> lower=-3.14 upper=3.14 effort=30 velocity=12
- joint left_shoulder_roll_joint: limit lower=-0.1745 upper=3.14 effort=10 velocity=10 -> lower=-0.1745 upper=3.14 effort=30 velocity=12
- joint left_shoulder_yaw_joint: limit lower=-3.14 upper=3.14 effort=10 velocity=10 -> lower=-3.14 upper=3.14 effort=30 velocity=12
- joint left_wrist_joint: limit lower=-3.14 upper=3.14 effort=10 velocity=10 -> lower=-3.14 upper=3.14 effort=30 velocity=12
- joint right_ankle_pitch_joint: limit lower=-0.6981 upper=0.5236 effort=10 velocity=10 -> lower=-0.6981 upper=0.5236 effort=30 velocity=12
- joint right_ankle_roll_joint: limit lower=-0.2618 upper=0.2618 effort=10 velocity=10 -> lower=-0.2618 upper=0.2618 effort=30 velocity=12
- joint right_elbow_joint: limit lower=-3.14 upper=1 effort=10 velocity=10 -> lower=-3.14 upper=1 effort=30 velocity=12
- joint right_hip_pitch_joint: limit lower=-2.862 upper=2.862 effort=10 velocity=10 -> lower=-2.862 upper=2.862 effort=120 velocity=25
- joint right_hip_roll_joint: limit lower=-2.6878 upper=0.1745 effort=10 velocity=10 -> lower=-2.6878 upper=0.1745 effort=120 velocity=25
- joint right_hip_yaw_joint: limit lower=-1.9199 upper=1.9199 effort=10 velocity=10 -> lower=-1.9199 upper=1.9199 effort=120 velocity=25
- joint right_knee_joint: limit lower=-0.2618 upper=2.7925 effort=10 velocity=10 -> lower=-0.2618 upper=2.7925 effort=120 velocity=25
- joint right_shoulder_pitch_joint: limit lower=-3.14 upper=3.14 effort=10 velocity=10 -> lower=-3.14 upper=3.14 effort=30 velocity=12
- joint right_shoulder_roll_joint: limit lower=-3.14 upper=0.1745 effort=10 velocity=10 -> lower=-3.14 upper=0.1745 effort=30 velocity=12
- joint right_shoulder_yaw_joint: limit lower=-3.14 upper=3.14 effort=10 velocity=10 -> lower=-3.14 upper=3.14 effort=30 velocity=12
- joint right_wrist_joint: limit lower=-3.14 upper=3.14 effort=10 velocity=10 -> lower=-3.14 upper=3.14 effort=30 velocity=12
- joint waist_roll_joint: limit lower=-0.7854 upper=0.7854 effort=10 velocity=10 -> lower=-0.7854 upper=0.7854 effort=120 velocity=25
- joint waist_yaw_joint: limit lower=-3.14 upper=3.14 effort=10 velocity=10 -> lower=-3.14 upper=3.14 effort=120 velocity=25

Commit message: fix collision

File: urdf/atom02.urdf (robot description, URDF)
Before this commit: robot atom02, 25 links, 24 joints
Links:
- link left_ankle_pitch_link: geometry visual mesh filename=../meshes/left_ankle_pitch_link_visual.stl
- link left_hip_pitch_link: geometry visual mesh filename=../meshes/left_hip_pitch_link_visual.stl
- link right_ankle_pitch_link: geometry visual mesh filename=../meshes/right_ankle_pitch_link_visual.stl
- link right_hip_pitch_link: geometry visual mesh filename=../meshes/right_hip_pitch_link_visual.stl
- link waist_roll_link: geometry visual mesh filename=../meshes/waist_roll_link_visual.stl

Commit message: update collision

File: urdf/atom02.urdf (robot description, URDF)
Before this commit: robot atom02, 25 links, 24 joints
Links:
- link left_ankle_roll_link: geometry collision sphere radius=0.005; collision sphere radius=0.005
- link right_ankle_roll_link: geometry collision sphere radius=0.005; collision sphere radius=0.005

Commit message: update collision

File: urdf/atom02.urdf (robot description, URDF)
Before this commit: robot atom02, 25 links, 24 joints
Links:
- link left_hip_pitch_link: geometry collision mesh filename=package://assets/merged/left_hip_pitch_link_collision.stl; visual mesh filename=../meshes/left_hip_pitch_link_visual.stl
- link right_hip_pitch_link: geometry collision mesh filename=../meshes/right_hip_pitch_link_collision.stl; visual mesh filename=../meshes/right_hip_pitch_link_visual.stl
- link waist_roll_link: geometry collision mesh filename=../meshes/waist_roll_link_collision.stl; visual mesh filename=../meshes/waist_roll_link_visual.stl

Commit message: fix bug

File: urdf/atom02.urdf (robot description, URDF)
Before this commit: robot atom02, 25 links, 24 joints
Links:
- link left_hip_pitch_link: geometry collision mesh filename=../meshes/left_hip_pitch_link_collision.stl; visual mesh filename=../meshes/left_hip_pitch_link_visual.stl
