Commit message: update urdf for rp1.2

File: urdf/rp1.urdf (robot description, URDF)
Before this commit: robot rp1, 25 links, 24 joints
Links:
- link base_link: mass 3.74331211 -> 3.587
- link left_ankle_pitch_link: mass 0.16959729 -> 0.174; geometry collision mesh filename=../meshes/left_ankle_pitch_link.STL; visual mesh filename=../meshes/left_ankle_pitch_link.STL
- link left_ankle_roll_link: mass 0.59697522 -> 0.788; geometry collision cylinder length=0.100 radius=0.005; collision cylinder length=0.100 radius=0.005
- link left_elbow_link: geometry collision mesh filename=../meshes/left_elbow_link.STL; visual mesh filename=../meshes/left_elbow_link.STL
- link left_hip_pitch_link: mass 1.69667825 -> 1.896; geometry collision mesh filename=../meshes/left_hip_pitch_link.STL; visual mesh filename=../meshes/left_hip_pitch_link.STL
- link left_hip_roll_link: mass 2.02732783 -> 1.758; geometry collision mesh filename=../meshes/left_hip_roll_link.STL; visual mesh filename=../meshes/left_hip_roll_link.STL
- link left_hip_yaw_link: mass 2.58081317 -> 2.584; geometry collision mesh filename=../meshes/left_hip_yaw_link.STL; visual mesh filename=../meshes/left_hip_yaw_link.STL
- link left_knee_link: mass 2.34293756 -> 3.004; geometry collision mesh filename=../meshes/left_knee_link.STL; visual mesh filename=../meshes/left_knee_link.STL
- link left_shoulder_pitch_link: geometry collision mesh filename=../meshes/left_shoulder_pitch_link.STL; visual mesh filename=../meshes/left_shoulder_pitch_link.STL
- link left_shoulder_roll_link: geometry visual mesh filename=../meshes/left_shoulder_roll_link.STL
- link left_shoulder_yaw_link: geometry collision mesh filename=../meshes/left_shoulder_yaw_link.STL; visual mesh filename=../meshes/left_shoulder_yaw_link.STL
- link left_wrist_link: geometry collision mesh filename=../meshes/left_wrist_link.STL; visual mesh filename=../meshes/left_wrist_link.STL
- link right_ankle_pitch_link: mass 0.16959729 -> 0.174; geometry collision mesh filename=../meshes/right_ankle_pitch_link.STL; visual mesh filename=../meshes/right_ankle_pitch_link.STL
- link right_ankle_roll_link: mass 0.59697522 -> 0.788; geometry collision cylinder length=0.100 radius=0.005; collision cylinder length=0.100 radius=0.005
- link right_elbow_link: geometry collision mesh filename=../meshes/right_elbow_link.STL; visual mesh filename=../meshes/right_elbow_link.STL
- link right_hip_pitch_link: mass 1.69667615 -> 1.896; geometry collision mesh filename=../meshes/right_hip_pitch_link.STL; visual mesh filename=../meshes/right_hip_pitch_link.STL
- link right_hip_roll_link: mass 2.01871347 -> 1.758; geometry collision mesh filename=../meshes/right_hip_roll_link.STL; visual mesh filename=../meshes/right_hip_roll_link.STL
- link right_hip_yaw_link: mass 2.58159271 -> 2.584; geometry collision mesh filename=../meshes/right_hip_yaw_link.STL; visual mesh filename=../meshes/right_hip_yaw_link.STL
- link right_knee_link: mass 2.34294346 -> 3.003; geometry collision mesh filename=../meshes/right_knee_link.STL; visual mesh filename=../meshes/right_knee_link.STL
- link right_shoulder_pitch_link: geometry collision mesh filename=../meshes/right_shoulder_pitch_link.STL; visual mesh filename=../meshes/right_shoulder_pitch_link.STL
- link right_shoulder_roll_link: geometry visual mesh filename=../meshes/right_shoulder_roll_link.STL
- link right_shoulder_yaw_link: mass 1.14691961 -> 0.90813471; geometry collision mesh filename=../meshes/right_shoulder_yaw_link.STL; visual mesh filename=../meshes/right_shoulder_yaw_link.STL
- link right_wrist_link: geometry collision mesh filename=../meshes/right_wrist_link.STL; visual mesh filename=../meshes/right_wrist_link.STL
- link waist_roll_link: mass 1.69337593 -> 1.738; geometry collision mesh filename=../meshes/waist_roll_link.STL; visual mesh filename=../meshes/waist_roll_link.STL
- link waist_yaw_link: geometry collision mesh filename=../meshes/waist_yaw_link.STL; visual mesh filename=../meshes/waist_yaw_link.STL
Joints:
- joint left_ankle_pitch_joint: limit lower=-0.69 upper=0.52 effort=20 velocity=8 -> lower=-0.78 upper=0.61 effort=28.5 velocity=20; origin xyz=-0.00139187168099175 0.0305005712971281 -0.304000157809516 rpy=0 0 0 -> xyz=0.03131 0.031809 -0.30533 rpy=0 0 0
- joint left_ankle_roll_joint: axis 1 0 0 -> 0.999993677858222 0 0.00355587451777954; limit lower=-0.26 upper=0.26 effort=20 velocity=8 -> lower=-0.26 upper=0.26 effort=28.5 velocity=20; origin xyz=0 0.00649999999999989 -0.018968626966597 rpy=0 0 0 -> xyz=6.75063037469253E-05 0 -0.0189998798792698 rpy=0 0 0
- joint left_elbow_joint: axis 0 1 0 -> 0 -1 0
- joint left_hip_pitch_joint: limit lower=-2.14 upper=2.14 effort=120 velocity=9 -> lower=-2.86 upper=2.86 effort=140 velocity=13.5; origin xyz=-0.0374249489846522 0.0724873458216877 -0.0557505673027586 rpy=0 0 0 -> xyz=-0.038429948015562 -0.0700126544457154 -0.0516391613039941 rpy=0 0 0
- joint left_hip_roll_joint: limit lower=-0.5 upper=3.5 effort=120 velocity=9 -> lower=-0.74 upper=2.6 effort=140 velocity=13.5; origin xyz=0.0306249999999995 0.0624994287029045 -0.0199999999999978 rpy=0 0 0 -> xyz=0.0329147207895102 0.194253937543099 -0.0606719292944441 rpy=0 0 0
- joint left_hip_yaw_joint: limit lower=-1.91 upper=1.91 effort=120 velocity=9 -> lower=-2.76 upper=2.76 effort=140 velocity=13.5; origin xyz=-0.0130381971475755 0 -0.137499999999989 rpy=0 0 0 -> xyz=-0.0136984138454024 0 -0.129000000000208 rpy=0 0 0
- joint left_knee_joint: limit lower=-2.86 upper=0.08 effort=120 velocity=9 -> lower=-2.83 upper=0.06 effort=140 velocity=13.5; origin xyz=-0.0309327936142636 -0.0370005712972284 -0.162502491489606 rpy=0 0 0 -> xyz=-0.0332010020225741 -0.0318089595042233 -0.165090361688273 rpy=0 0 0
- joint right_ankle_pitch_joint: limit lower=-0.69 upper=0.52 effort=20 velocity=8 -> lower=-0.78 upper=0.61 effort=28.5 velocity=20; origin xyz=-0.00139187168099966 -0.0370005712971978 -0.304000157809505 rpy=0 0 0 -> xyz=0.0313104411691826 -0.0318089580741854 -0.305328803190489 rpy=0 0 0
- joint right_ankle_roll_joint: axis 1 0 0 -> 0.999993677858222 0 0.00355587451777984; limit lower=-0.26 upper=0.26 effort=20 velocity=8 -> lower=-0.26 upper=0.26 effort=28.5 velocity=20; origin xyz=0 0 -0.018968626966597 rpy=0 0 0 -> xyz=6.75616158378675E-05 0 -0.0189998798793065 rpy=0 0 0
- joint right_elbow_joint: axis 0 -1 0 -> 0 1 0
- joint right_hip_pitch_joint: limit lower=-2.14 upper=2.14 effort=120 velocity=9 -> lower=-2.86 upper=2.86 effort=140 velocity=13.5; origin xyz=-0.03742444898466 -0.0675126541783108 -0.0557505673027595 rpy=0 0 0 -> xyz=-0.03843 0.063987 -0.051639 rpy=0 0 0
- joint right_hip_roll_joint: limit lower=-3.5 upper=0.5 effort=120 velocity=9 -> lower=-2.6 upper=0.74 effort=140 velocity=13.5; origin xyz=0.0306245000000074 -0.0625 -0.0200000000000002 rpy=0 0 0 -> xyz=0.037924 -0.19425 -0.060672 rpy=0 0 0
- joint right_hip_yaw_joint: limit lower=-1.91 upper=1.91 effort=120 velocity=9 -> lower=-2.76 upper=2.76 effort=140 velocity=13.5; origin xyz=-0.0130381971463119 0 -0.1375 rpy=0 0 0 -> xyz=-0.0187081031828124 0 -0.129 rpy=0 0 0
- joint right_knee_joint: limit lower=-0.08 upper=2.86 effort=120 velocity=9 -> lower=-0.06 upper=2.83 effort=140 velocity=13.5; origin xyz=-0.0309327936155297 0.037 -0.1625024914896 rpy=0 0 0 -> xyz=-0.033201 0.031809 -0.16509 rpy=0 0 0
- joint waist_roll_joint: limit lower=-0.69 upper=0.69 effort=120 velocity=9 -> lower=-0.7 upper=0.7 effort=140 velocity=13.5; origin xyz=-0.00679994881842894 0.00248734582169075 0.0492495461463824 rpy=0 0 0 -> xyz=-0.0065799 -0.0030127 0.052984 rpy=0 0 0
- joint waist_yaw_joint: limit lower=-2.26 upper=3.32 effort=120 velocity=9 -> lower=-2.26 upper=3.32 effort=140 velocity=13.5

Commit message: update limits

File: urdf/rp1.urdf (robot description, URDF)
Before this commit: robot rp1.2, 25 links, 24 joints
Joints:
- joint left_elbow_joint: limit lower=-1.1 upper=1.7 effort=20 velocity=8 -> lower=-1.7 upper=1.1 effort=20 velocity=8
- joint right_elbow_joint: limit lower=-1.7 upper=1.1 effort=20 velocity=8 -> lower=-1.1 upper=1.7 effort=20 velocity=8

Commit message: update urdf for rp1.3

File: urdf/rp1.urdf (robot description, URDF)
Before this commit: robot rp1.2, 25 links, 24 joints
Links:
- added link left_wrist_pitch_link, mass 1.1081; collision mesh filename=../meshes/left_wrist_pitch_link.STL; visual mesh filename=../meshes/left_wrist_pitch_link.STL
- added link left_wrist_roll_link, mass 0.0732; collision mesh filename=../meshes/left_wrist_roll_link.STL; visual mesh filename=../meshes/left_wrist_roll_link.STL
- added link right_wrist_pitch_link, mass 1.1083; collision mesh filename=../meshes/right_wrist_pitch_link.STL; visual mesh filename=../meshes/right_wrist_pitch_link.STL
- added link right_wrist_roll_link, mass 0.0732; collision mesh filename=../meshes/right_wrist_roll_link.STL; visual mesh filename=../meshes/right_wrist_roll_link.STL
- link base_link: mass 3.587 -> 3.5521
- link left_ankle_pitch_link: mass 0.174 -> 0.1661
- link left_ankle_roll_link: mass 0.788 -> 0.7882
- link left_elbow_link: mass 0.74855627 -> 0.8177
- link left_hip_pitch_link: mass 1.896 -> 1.8622
- link left_hip_roll_link: mass 1.758 -> 1.7439
- link left_hip_yaw_link: mass 2.584 -> 2.5702
- link left_knee_link: mass 3.004 -> 2.7678
- link left_shoulder_pitch_link: mass 0.64909166 -> 0.7655
- link left_shoulder_roll_link: mass 0.68815424 -> 0.8044; geometry collision mesh filename=../meshes/left_shoulder_roll_link.STL; visual mesh filename=../meshes/left_shoulder_roll_link.STL
- link left_shoulder_yaw_link: mass 0.90825302 -> 1.1046
- link left_wrist_link: mass 0.17378226 -> 0.1588
- link right_ankle_pitch_link: mass 0.174 -> 0.1661
- link right_ankle_roll_link: mass 0.788 -> 0.7882
- link right_elbow_link: mass 0.74855589 -> 0.8174
- link right_hip_pitch_link: mass 1.896 -> 1.8622
- link right_hip_roll_link: mass 1.758 -> 1.7439
- link right_hip_yaw_link: mass 2.584 -> 2.5701
- link right_knee_link: mass 3.003 -> 2.7871
- link right_shoulder_pitch_link: mass 0.65011229 -> 0.7953
- link right_shoulder_roll_link: mass 0.69111022 -> 0.8044; geometry collision mesh filename=../meshes/right_shoulder_roll_link.STL; visual mesh filename=../meshes/right_shoulder_roll_link.STL
- link right_shoulder_yaw_link: mass 0.90813471 -> 1.0884
- link right_wrist_link: mass 0.21895422 -> 0.1588
- link waist_roll_link: mass 1.738 -> 1.8289
- link waist_yaw_link: mass 5.79223222 -> 7.5258
Joints:
- added joint left_wrist_pitch_joint: type revolute, parent left_wrist_link, child left_wrist_pitch_link, origin xyz=0.053 0.020701 0 rpy=0 0 0, axis 0 1 0, limit lower=-1.4 upper=1.4 effort=20 velocity=8
- added joint left_wrist_roll_joint: type revolute, parent left_wrist_pitch_link, child left_wrist_roll_link, origin xyz=0.062136 -0.02585 0.029075 rpy=0 0 0, axis 0 0 1, limit lower=-1.22 upper=1.22 effort=20 velocity=8
- added joint right_wrist_pitch_joint: type revolute, parent right_wrist_link, child right_wrist_pitch_link, origin xyz=0.045 -0.020701 0 rpy=0 0 0, axis 0 -1 0, limit lower=-1.4 upper=1.4 effort=20 velocity=8
- added joint right_wrist_roll_joint: type revolute, parent right_wrist_pitch_link, child right_wrist_roll_link, origin xyz=0.062136 0.025685 0.029241 rpy=0 0 0, axis 0 0 1, limit lower=-1.22 upper=1.22 effort=20 velocity=8
- joint left_ankle_pitch_joint: origin xyz=0.03131 0.031809 -0.30533 rpy=0 0 0 -> xyz=0.03131 0.031811 -0.30533 rpy=0 0 0
- joint left_ankle_roll_joint: origin xyz=6.75063037469253E-05 0 -0.0189998798792698 rpy=0 0 0 -> xyz=0.013067 0 -0.018922 rpy=0 0 0
- joint left_elbow_joint: limit lower=-1.7 upper=1.1 effort=20 velocity=8 -> lower=-1.6 upper=1.24 effort=20 velocity=8; origin xyz=0.0094386 -0.027125 -0.12693 rpy=0 0 0 -> xyz=0.020793 -0.031888 -0.10414 rpy=0 0 0
- joint left_hip_pitch_joint: origin xyz=-0.038429948015562 -0.0700126544457154 -0.0516391613039941 rpy=0 0 0 -> xyz=-0.03843 0.063987 -0.051639 rpy=0 0 0
- joint left_hip_roll_joint: origin xyz=0.0329147207895102 0.194253937543099 -0.0606719292944441 rpy=0 0 0 -> xyz=0.032915 0.060254 -0.060672 rpy=0 0 0
- joint left_hip_yaw_joint: origin xyz=-0.0136984138454024 0 -0.129000000000208 rpy=0 0 0 -> xyz=-0.013698 0 -0.129 rpy=0 0 0
- joint left_knee_joint: origin xyz=-0.0332010020225741 -0.0318089595042233 -0.165090361688273 rpy=0 0 0 -> xyz=-0.033201 -0.031809 -0.16509 rpy=0 0 0
- joint left_shoulder_pitch_joint: axis 0 1 0 -> 0 0.99619 0.087156; limit lower=-2.7 upper=2.7 effort=20 velocity=8 -> lower=-3.4 upper=2.35 effort=20 velocity=8; origin xyz=-0.00499999999999793 0.10137354822811 0.203401111781171 rpy=0.0436332312998421 0 0 -> xyz=-0.0035001 0.11385 0.19939 rpy=0 0 0
- joint left_shoulder_roll_joint: axis -1 0 0 -> 1 0 0; limit lower=-2.89 upper=0.26 effort=20 velocity=8 -> lower=-0.47 upper=2.9 effort=20 velocity=8; origin xyz=-0.027722 0.0607 0 rpy=-0.043633 0 0 -> xyz=0.028402 0.060357 -0.015009 rpy=0 0 0
- joint left_shoulder_yaw_joint: limit lower=-2.7 upper=2.7 effort=20 velocity=8 -> lower=-2.87 upper=2.87 effort=20 velocity=8; origin xyz=0.0276538600051183 0.00647148427864618 -0.103006241732382 rpy=0 0 0 -> xyz=-0.019058 0 -0.105 rpy=0 0 0
- joint left_wrist_joint: limit lower=-2.7 upper=2.7 effort=20 velocity=8 -> lower=-2.56 upper=2.56 effort=20 velocity=8; origin xyz=0.105895445525297 0.0272010393332496 -0.0134505488341287 rpy=0 0 0 -> xyz=0.11609 0.031859 -0.018793 rpy=0 0 0
- joint right_ankle_pitch_joint: origin xyz=0.0313104411691826 -0.0318089580741854 -0.305328803190489 rpy=0 0 0 -> xyz=0.03131 -0.031809 -0.30533 rpy=0 0 0
- joint right_ankle_roll_joint: origin xyz=6.75616158378675E-05 0 -0.0189998798793065 rpy=0 0 0 -> xyz=0.013067 0 -0.018922 rpy=0 0 0
- joint right_elbow_joint: limit lower=-1.1 upper=1.7 effort=20 velocity=8 -> lower=-1.24 upper=1.6 effort=20 velocity=8; origin xyz=0.0094385 0.027125 -0.12693 rpy=0 0 0 -> xyz=0.020793 0.031888 -0.10414 rpy=0 0 0
- joint right_hip_pitch_joint: origin xyz=-0.03843 0.063987 -0.051639 rpy=0 0 0 -> xyz=-0.03843 -0.070013 -0.051639 rpy=0 0 0
- joint right_hip_roll_joint: origin xyz=0.037924 -0.19425 -0.060672 rpy=0 0 0 -> xyz=0.032915 -0.060254 -0.060672 rpy=0 0 0
- joint right_hip_yaw_joint: origin xyz=-0.0187081031828124 0 -0.129 rpy=0 0 0 -> xyz=-0.013698 0 -0.129 rpy=0 0 0
- joint right_shoulder_pitch_joint: axis 0 -1 0 -> 0 -0.99619 0.087156; limit lower=-2.7 upper=2.7 effort=20 velocity=8 -> lower=-2.35 upper=3.4 effort=20 velocity=8; origin xyz=-0.00499999999999993 -0.101373548228108 0.203401111781173 rpy=-0.0436332312998597 0 0 -> xyz=-0.0035 -0.11385 0.19939 rpy=0 0 0
- joint right_shoulder_roll_joint: axis -1 0 0 -> 1 0 0; limit lower=-0.26 upper=2.89 effort=20 velocity=8 -> lower=-2.9 upper=0.47 effort=20 velocity=8; origin xyz=-0.027528 -0.060704 9.1336E-05 rpy=0.043633 0 0 -> xyz=0.028402 -0.060357 -0.015009 rpy=0 0 0
- joint right_shoulder_yaw_joint: limit lower=-2.7 upper=2.7 effort=20 velocity=8 -> lower=-2.87 upper=2.87 effort=20 velocity=8; origin xyz=0.0276538600055591 -0.00647148427843708 -0.103006241732399 rpy=0 0 0 -> xyz=-0.019058 0 -0.105 rpy=0 0 0
- joint right_wrist_joint: limit lower=-2.7 upper=2.7 effort=20 velocity=8 -> lower=-2.56 upper=2.56 effort=20 velocity=8; origin xyz=0.105895321727716 -0.0272010056651584 -0.0134515915317502 rpy=0 0 0 -> xyz=0.11609 -0.031859 -0.018793 rpy=0 0 0
- joint waist_roll_joint: origin xyz=-0.0065799 -0.0030127 0.052984 rpy=0 0 0 -> xyz=-0.0065899 -0.0030127 0.052984 rpy=0 0 0
- joint waist_yaw_joint: limit lower=-2.26 upper=3.32 effort=140 velocity=13.5 -> lower=-2.91 upper=2.91 effort=140 velocity=13.5; origin xyz=-0.0303363545807988 0 0.0617500000001175 rpy=0 0 0 -> xyz=-0.031845 0 0.067 rpy=0 0 0

Commit message: fix bug

File: urdf/rp1.urdf (robot description, URDF)
Before this commit: robot rp1.3.1, 29 links, 28 joints
Links:
- removed link left_wrist_link
- removed link right_wrist_link
- added link left_wrist_yaw_link, mass 0.0732; collision mesh filename=../meshes/left_wrist_yaw_link.STL; visual mesh filename=../meshes/left_wrist_yaw_link.STL
- added link right_wrist_yaw_link, mass 0.0732; collision mesh filename=../meshes/right_wrist_yaw_link.STL; visual mesh filename=../meshes/right_wrist_yaw_link.STL
- link left_wrist_roll_link: mass 0.0732 -> 0.1588
- link right_wrist_roll_link: mass 0.0732 -> 0.1588
Joints:
- removed joint left_wrist_joint
- removed joint right_wrist_joint
- added joint left_wrist_yaw_joint: type revolute, parent left_wrist_pitch_link, child left_wrist_yaw_link, origin xyz=0.062136 -0.02585 0.029075 rpy=0 0 0, axis 0 0 1, limit lower=-1.22 upper=1.22 effort=20 velocity=8
- added joint right_wrist_yaw_joint: type revolute, parent right_wrist_pitch_link, child right_wrist_yaw_link, origin xyz=0.062136 0.025685 0.029241 rpy=0 0 0, axis 0 0 1, limit lower=-1.22 upper=1.22 effort=20 velocity=8
- joint left_wrist_pitch_joint: axis 0 1 0 -> 0 -1 0; parent left_wrist_link -> left_wrist_roll_link
- joint left_wrist_roll_joint: axis 0 0 1 -> 1 0 0; limit lower=-1.22 upper=1.22 effort=20 velocity=8 -> lower=-2.56 upper=2.56 effort=20 velocity=8; origin xyz=0.062136 -0.02585 0.029075 rpy=0 0 0 -> xyz=0.11609 0.031859 -0.018793 rpy=0 0 0; parent left_wrist_pitch_link -> left_elbow_link
- joint right_wrist_pitch_joint: axis 0 -1 0 -> 0 1 0; parent right_wrist_link -> right_wrist_roll_link
- joint right_wrist_roll_joint: axis 0 0 1 -> 1 0 0; limit lower=-1.22 upper=1.22 effort=20 velocity=8 -> lower=-2.56 upper=2.56 effort=20 velocity=8; origin xyz=0.062136 0.025685 0.029241 rpy=0 0 0 -> xyz=0.11609 -0.031859 -0.018793 rpy=0 0 0; parent right_wrist_pitch_link -> right_elbow_link

Commit message: update wrist link

File: urdf/rp1.urdf (robot description, URDF)
Before this commit: robot rp1.3.1, 29 links, 28 joints
Links:
- link base_link: mass 3.5521 -> 3.55209336
- link left_ankle_pitch_link: mass 0.1661 -> 0.17366118
- link left_ankle_roll_link: mass 0.7882 -> 0.78817642
- link left_elbow_link: mass 0.8177 -> 0.81770364
- link left_hip_pitch_link: mass 1.8622 -> 1.86216378
- link left_hip_roll_link: mass 1.7439 -> 1.74387104
- link left_hip_yaw_link: mass 2.5702 -> 2.57015343
- link left_knee_link: mass 2.7678 -> 2.78730161
- link left_shoulder_pitch_link: mass 0.7655 -> 0.79513665
- link left_shoulder_roll_link: mass 0.8044 -> 0.80442734
- link left_shoulder_yaw_link: mass 1.1046 -> 1.10463444
- link left_wrist_pitch_link: mass 1.1081 -> 0.07319805
- link left_wrist_roll_link: mass 0.1588 -> 0.15878030
- link left_wrist_yaw_link: mass 0.0732 -> 1.10833884
- link right_ankle_pitch_link: mass 0.1661 -> 0.17366118
- link right_ankle_roll_link: mass 0.7882 -> 0.78817642
- link right_elbow_link: mass 0.8174 -> 0.81744969
- link right_hip_pitch_link: mass 1.8622 -> 1.86219733
- link right_hip_roll_link: mass 1.7439 -> 1.74387104
- link right_hip_yaw_link: mass 2.5701 -> 2.57008707
- link right_knee_link: mass 2.7871 -> 2.78711852
- link right_shoulder_pitch_link: mass 0.7953 -> 0.79525140
- link right_shoulder_roll_link: mass 0.8044 -> 0.80442734
- link right_shoulder_yaw_link: mass 1.0884 -> 1.08841996
- link right_wrist_pitch_link: mass 1.1083 -> 0.07319805
- link right_wrist_roll_link: mass 0.1588 -> 0.15878030
- link right_wrist_yaw_link: mass 0.0732 -> 1.10814793
- link waist_roll_link: mass 1.8289 -> 1.82887777
- link waist_yaw_link: mass 7.5258 -> 7.52582874
Joints:
- joint left_wrist_pitch_joint: axis 0 -1 0 -> 0 1 0; limit lower=-1.4 upper=1.4 effort=20 velocity=8 -> lower=-1.22 upper=1.22 effort=20 velocity=8; origin xyz=0.053 0.020701 0 rpy=0 0 0 -> xyz=0.062136 0.029241 -0.025685 rpy=0 0 0; parent left_wrist_roll_link -> left_wrist_yaw_link
- joint left_wrist_yaw_joint: axis 0 0 1 -> 0 0 -1; origin xyz=0.062136 -0.02585 0.029075 rpy=0 0 0 -> xyz=0.053 0 0.020701 rpy=0 0 0; parent left_wrist_pitch_link -> left_wrist_roll_link
- joint right_wrist_pitch_joint: axis 0 1 0 -> 0 -1 0; limit lower=-1.4 upper=1.4 effort=20 velocity=8 -> lower=-1.22 upper=1.22 effort=20 velocity=8; origin xyz=0.045 -0.020701 0 rpy=0 0 0 -> xyz=0.062136 -0.029075 -0.02585 rpy=0 0 0; parent right_wrist_roll_link -> right_wrist_yaw_link
- joint right_wrist_yaw_joint: axis 0 0 1 -> 0 0 -1; origin xyz=0.062136 0.025685 0.029241 rpy=0 0 0 -> xyz=0.053 0 0.020701 rpy=0 0 0; parent right_wrist_pitch_link -> right_wrist_roll_link

Commit message: update actuator

File: urdf/rp1.urdf (robot description, URDF)
Before this commit: robot rp1.3.1, 29 links, 28 joints
Joints:
- joint left_ankle_pitch_joint: limit lower=-0.78 upper=0.61 effort=28.5 velocity=20 -> lower=-0.78 upper=0.61 effort=57 velocity=20
- joint left_ankle_roll_joint: limit lower=-0.26 upper=0.26 effort=28.5 velocity=20 -> lower=-0.26 upper=0.26 effort=57 velocity=20
- joint left_elbow_joint: limit lower=-1.6 upper=1.24 effort=20 velocity=8 -> lower=-1.6 upper=1.24 effort=28.5 velocity=20
- joint left_shoulder_pitch_joint: limit lower=-3.4 upper=2.35 effort=20 velocity=8 -> lower=-3.4 upper=2.35 effort=28.5 velocity=20
- joint left_shoulder_roll_joint: limit lower=-0.47 upper=2.9 effort=20 velocity=8 -> lower=-0.47 upper=2.9 effort=28.5 velocity=20
- joint left_shoulder_yaw_joint: limit lower=-2.87 upper=2.87 effort=20 velocity=8 -> lower=-2.87 upper=2.87 effort=28.5 velocity=20
- joint left_wrist_pitch_joint: limit lower=-1.22 upper=1.22 effort=20 velocity=8 -> lower=-1.22 upper=1.22 effort=28.5 velocity=20
- joint left_wrist_roll_joint: limit lower=-2.56 upper=2.56 effort=20 velocity=8 -> lower=-2.56 upper=2.56 effort=28.5 velocity=20
- joint left_wrist_yaw_joint: limit lower=-1.22 upper=1.22 effort=20 velocity=8 -> lower=-1.22 upper=1.22 effort=28.5 velocity=20
- joint right_ankle_pitch_joint: limit lower=-0.78 upper=0.61 effort=28.5 velocity=20 -> lower=-0.78 upper=0.61 effort=57 velocity=20
- joint right_ankle_roll_joint: limit lower=-0.26 upper=0.26 effort=28.5 velocity=20 -> lower=-0.26 upper=0.26 effort=57 velocity=20
- joint right_elbow_joint: limit lower=-1.24 upper=1.6 effort=20 velocity=8 -> lower=-1.24 upper=1.6 effort=28.5 velocity=20
- joint right_shoulder_pitch_joint: limit lower=-2.35 upper=3.4 effort=20 velocity=8 -> lower=-2.35 upper=3.4 effort=28.5 velocity=20
- joint right_shoulder_roll_joint: limit lower=-2.9 upper=0.47 effort=20 velocity=8 -> lower=-2.9 upper=0.47 effort=28.5 velocity=20
- joint right_shoulder_yaw_joint: limit lower=-2.87 upper=2.87 effort=20 velocity=8 -> lower=-2.87 upper=2.87 effort=28.5 velocity=20
- joint right_wrist_pitch_joint: limit lower=-1.22 upper=1.22 effort=20 velocity=8 -> lower=-1.22 upper=1.22 effort=28.5 velocity=20
- joint right_wrist_roll_joint: limit lower=-2.56 upper=2.56 effort=20 velocity=8 -> lower=-2.56 upper=2.56 effort=28.5 velocity=20
- joint right_wrist_yaw_joint: limit lower=-1.22 upper=1.22 effort=20 velocity=8 -> lower=-1.22 upper=1.22 effort=28.5 velocity=20
