Commit message: update limits

File: urdf/rp1.urdf (robot description, URDF)
Before this commit: robot rp1.3.1, 29 links, 28 joints
Joints:
- joint left_ankle_pitch_joint: limit lower=-0.78 upper=0.61 effort=57 velocity=20 -> lower=-0.78 upper=0.61 effort=70.6 velocity=21.88648
- joint left_ankle_roll_joint: limit lower=-0.26 upper=0.26 effort=57 velocity=20 -> lower=-0.26 upper=0.26 effort=70.6 velocity=21.88648
- joint left_elbow_joint: limit lower=-1.6 upper=1.24 effort=28.5 velocity=20 -> lower=-1.6 upper=1.24 effort=35.3 velocity=21.88648
- joint left_hip_pitch_joint: limit lower=-2.86 upper=2.86 effort=140 velocity=13.5 -> lower=-2.86 upper=2.86 effort=141.7 velocity=14.24192
- joint left_hip_roll_joint: limit lower=-0.74 upper=2.6 effort=140 velocity=13.5 -> lower=-0.74 upper=2.6 effort=141.7 velocity=14.24192
- joint left_hip_yaw_joint: limit lower=-2.76 upper=2.76 effort=140 velocity=13.5 -> lower=-2.76 upper=2.76 effort=141.7 velocity=14.24192
- joint left_knee_joint: limit lower=-2.83 upper=0.06 effort=140 velocity=13.5 -> lower=-2.83 upper=0.06 effort=141.7 velocity=14.24192
- joint left_shoulder_pitch_joint: limit lower=-3.4 upper=2.35 effort=28.5 velocity=20 -> lower=-3.4 upper=2.35 effort=35.3 velocity=21.88648
- joint left_shoulder_roll_joint: limit lower=-0.47 upper=2.9 effort=28.5 velocity=20 -> lower=-0.47 upper=2.9 effort=35.3 velocity=21.88648
- joint left_shoulder_yaw_joint: limit lower=-2.87 upper=2.87 effort=28.5 velocity=20 -> lower=-2.87 upper=2.87 effort=35.3 velocity=21.88648
- joint left_wrist_pitch_joint: limit lower=-1.22 upper=1.22 effort=28.5 velocity=20 -> lower=-1.22 upper=1.22 effort=35.3 velocity=21.88648
- joint left_wrist_roll_joint: limit lower=-2.56 upper=2.56 effort=28.5 velocity=20 -> lower=-2.56 upper=2.56 effort=35.3 velocity=21.88648
- joint left_wrist_yaw_joint: limit lower=-1.22 upper=1.22 effort=28.5 velocity=20 -> lower=-1.22 upper=1.22 effort=35.3 velocity=21.88648
- joint right_ankle_pitch_joint: limit lower=-0.78 upper=0.61 effort=57 velocity=20 -> lower=-0.78 upper=0.61 effort=70.6 velocity=21.88648
- joint right_ankle_roll_joint: limit lower=-0.26 upper=0.26 effort=57 velocity=20 -> lower=-0.26 upper=0.26 effort=70.6 velocity=21.88648
- joint right_elbow_joint: limit lower=-1.24 upper=1.6 effort=28.5 velocity=20 -> lower=-1.24 upper=1.6 effort=35.3 velocity=21.88648
- joint right_hip_pitch_joint: limit lower=-2.86 upper=2.86 effort=140 velocity=13.5 -> lower=-2.86 upper=2.86 effort=141.7 velocity=14.24192
- joint right_hip_roll_joint: limit lower=-2.6 upper=0.74 effort=140 velocity=13.5 -> lower=-2.6 upper=0.74 effort=141.7 velocity=14.24192
- joint right_hip_yaw_joint: limit lower=-2.76 upper=2.76 effort=140 velocity=13.5 -> lower=-2.76 upper=2.76 effort=141.7 velocity=14.24192
- joint right_knee_joint: limit lower=-0.06 upper=2.83 effort=140 velocity=13.5 -> lower=-0.06 upper=2.83 effort=141.7 velocity=14.24192
- joint right_shoulder_pitch_joint: limit lower=-2.35 upper=3.4 effort=28.5 velocity=20 -> lower=-2.35 upper=3.4 effort=35.3 velocity=21.88648
- joint right_shoulder_roll_joint: limit lower=-2.9 upper=0.47 effort=28.5 velocity=20 -> lower=-2.9 upper=0.47 effort=35.3 velocity=21.88648
- joint right_shoulder_yaw_joint: limit lower=-2.87 upper=2.87 effort=28.5 velocity=20 -> lower=-2.87 upper=2.87 effort=35.3 velocity=21.88648
- joint right_wrist_pitch_joint: limit lower=-1.22 upper=1.22 effort=28.5 velocity=20 -> lower=-1.22 upper=1.22 effort=35.3 velocity=21.88648
- joint right_wrist_roll_joint: limit lower=-2.56 upper=2.56 effort=28.5 velocity=20 -> lower=-2.56 upper=2.56 effort=35.3 velocity=21.88648
- joint right_wrist_yaw_joint: limit lower=-1.22 upper=1.22 effort=28.5 velocity=20 -> lower=-1.22 upper=1.22 effort=35.3 velocity=21.88648
- joint waist_roll_joint: limit lower=-0.7 upper=0.7 effort=140 velocity=13.5 -> lower=-0.7 upper=0.7 effort=141.7 velocity=14.24192
- joint waist_yaw_joint: limit lower=-2.91 upper=2.91 effort=140 velocity=13.5 -> lower=-2.91 upper=2.91 effort=141.7 velocity=14.24192

Commit message: update rp1.3.1

File: urdf/rp1.urdf (robot description, URDF)
Before this commit: robot rp1.3.1, 29 links, 28 joints
Links:
- link left_shoulder_pitch_link: mass 0.79513665 -> 0.83889911
- link left_shoulder_yaw_link: mass 1.10463444 -> 1.10463437
- link right_shoulder_pitch_link: mass 0.79525140 -> 0.83890716
- link waist_yaw_link: mass 7.52582874 -> 8.02130808
Joints:
- joint left_shoulder_pitch_joint: origin xyz=-0.0035001 0.11385 0.19939 rpy=0 0 0 -> xyz=0 0.1165 0.19949 rpy=0 0 0
- joint right_shoulder_pitch_joint: origin xyz=-0.0035 -0.11385 0.19939 rpy=0 0 0 -> xyz=0 -0.1165 0.19949 rpy=0 0 0
