Commit message: update rp1.3.2

File: urdf/rp1.urdf (robot description, URDF)
Before this commit: robot rp1.3.1, 29 links, 28 joints
Links:
- link base_link: mass 3.55209336 -> 3.23587253
- link left_ankle_pitch_link: mass 0.17366118 -> 0.16605731
- link left_ankle_roll_link: mass 0.78817642 -> 0.71237841
- link left_elbow_link: mass 0.81770364 -> 0.77922872
- link left_hip_pitch_link: mass 1.86216378 -> 1.83930168
- link left_hip_roll_link: mass 1.74387104 -> 1.45932598
- link left_hip_yaw_link: mass 2.57015343 -> 2.38381463
- link left_knee_link: mass 2.78730161 -> 2.45769202
- link left_shoulder_pitch_link: mass 0.83889911 -> 0.82850012
- link left_shoulder_roll_link: mass 0.80442734 -> 0.76916758
- link left_shoulder_yaw_link: mass 1.10463437 -> 0.95227320
- link left_wrist_roll_link: mass 0.15878030 -> 0.16115938
- link left_wrist_yaw_link: mass 1.10833884 -> 1.03494219
- link right_ankle_pitch_link: mass 0.17366118 -> 0.16605731
- link right_ankle_roll_link: mass 0.78817642 -> 0.71237841
- link right_elbow_link: mass 0.81744969 -> 0.77922499
- link right_hip_pitch_link: mass 1.86219733 -> 1.84174869
- link right_hip_roll_link: mass 1.74387104 -> 1.45932598
- link right_hip_yaw_link: mass 2.57008707 -> 2.38427565
- link right_knee_link: mass 2.78711852 -> 2.44960559
- link right_shoulder_pitch_link: mass 0.83890716 -> 0.82850796
- link right_shoulder_yaw_link: mass 1.08841996 -> 0.95225273
- link right_wrist_pitch_link: mass 0.07319805 -> 0.07221264
- link right_wrist_roll_link: mass 0.15878030 -> 0.16115938
- link right_wrist_yaw_link: mass 1.10814793 -> 1.03493727
- link waist_roll_link: mass 1.82887777 -> 1.53201882
- link waist_yaw_link: mass 8.02130808 -> 7.53658565
Joints:
- joint left_ankle_pitch_joint: origin xyz=0.03131 0.031811 -0.30533 rpy=0 0 0 -> xyz=0.03131 0.030811 -0.30533 rpy=0 0 0
- joint left_elbow_joint: origin xyz=0.020793 -0.031888 -0.10414 rpy=0 0 0 -> xyz=0.020796 -0.031888 -0.10414 rpy=0 0 0
- joint left_hip_pitch_joint: origin xyz=-0.03843 0.063987 -0.051639 rpy=0 0 0 -> xyz=-0.03843 0.062987 -0.051639 rpy=0 0 0
- joint left_hip_roll_joint: origin xyz=0.032915 0.060254 -0.060672 rpy=0 0 0 -> xyz=0.031915 0.061254 -0.060672 rpy=0 0 0
- joint left_hip_yaw_joint: origin xyz=-0.013698 0 -0.129 rpy=0 0 0 -> xyz=-0.012698 0 -0.129 rpy=0 0 0
- joint left_knee_joint: origin xyz=-0.033201 -0.031809 -0.16509 rpy=0 0 0 -> xyz=-0.033201 -0.030809 -0.16509 rpy=0 0 0
- joint left_shoulder_pitch_joint: origin xyz=0 0.1165 0.19949 rpy=0 0 0 -> xyz=0 0.116496194698121 0.19848715574272 rpy=0 0 0
- joint left_shoulder_roll_joint: origin xyz=0.028402 0.060357 -0.015009 rpy=0 0 0 -> xyz=0.0287432951006891 0.0653494445514435 -0.014608906526987 rpy=0 0 0
- joint left_shoulder_yaw_joint: origin xyz=-0.019058 0 -0.105 rpy=0 0 0 -> xyz=-0.0190574930004302 0 -0.105000039994097 rpy=0 0 0
- joint left_wrist_pitch_joint: origin xyz=0.062136 0.029241 -0.025685 rpy=0 0 0 -> xyz=0.062136 0.029458 -0.026067 rpy=0 0 0
- joint left_wrist_roll_joint: origin xyz=0.11609 0.031859 -0.018793 rpy=0 0 0 -> xyz=0.116093381994033 0.031859446289993 -0.0187927584979322 rpy=0 0 0
- joint right_ankle_pitch_joint: origin xyz=0.03131 -0.031809 -0.30533 rpy=0 0 0 -> xyz=0.03131 -0.030809 -0.30533 rpy=0 0 0
- joint right_elbow_joint: origin xyz=0.020793 0.031888 -0.10414 rpy=0 0 0 -> xyz=0.0207956801502895 0.031887525882762 -0.104135222723484 rpy=0 0 0
- joint right_hip_pitch_joint: origin xyz=-0.03843 -0.070013 -0.051639 rpy=0 0 0 -> xyz=-0.03843 -0.069013 -0.051639 rpy=0 0 0
- joint right_hip_roll_joint: origin xyz=0.032915 -0.060254 -0.060672 rpy=0 0 0 -> xyz=0.031915 -0.061254 -0.060672 rpy=0 0 0
- joint right_hip_yaw_joint: origin xyz=-0.013698 0 -0.129 rpy=0 0 0 -> xyz=-0.012698 0 -0.129 rpy=0 0 0
- joint right_knee_joint: origin xyz=-0.033201 0.031809 -0.16509 rpy=0 0 0 -> xyz=-0.0332010004232152 0.0308089665012395 -0.165090022909223 rpy=0 0 0
- joint right_shoulder_pitch_joint: origin xyz=0 -0.1165 0.19949 rpy=0 0 0 -> xyz=0 -0.116496194698064 0.198487155742749 rpy=0 0 0
- joint right_shoulder_roll_joint: origin xyz=0.028402 -0.060357 -0.015009 rpy=0 0 0 -> xyz=0.0287432951007422 -0.0653494445235536 -0.0146089065305009 rpy=0 0 0
- joint right_shoulder_yaw_joint: origin xyz=-0.019058 0 -0.105 rpy=0 0 0 -> xyz=-0.0190573923593691 0 -0.105000126276637 rpy=0 0 0
- joint right_wrist_pitch_joint: origin xyz=0.062136 -0.029075 -0.02585 rpy=0 0 0 -> xyz=0.062136 -0.029458 -0.026067 rpy=0 0 0
- joint right_wrist_roll_joint: origin xyz=0.11609 -0.031859 -0.018793 rpy=0 0 0 -> xyz=0.11609334409225 -0.031859369715491 -0.0187927299688337 rpy=0 0 0
- joint waist_roll_joint: origin xyz=-0.0065899 -0.0030127 0.052984 rpy=0 0 0 -> xyz=-0.00757994881845658 -0.00301269924435144 0.0529838303646947 rpy=0 0 0
- joint waist_yaw_joint: origin xyz=-0.031845 0 0.067 rpy=0 0 0 -> xyz=-0.0308449999997339 0 0.0679999999997294 rpy=0 0 0

File: urdf/rp1_24dof.urdf (robot description, URDF)
Before this commit: robot rp1.3.1, 25 links, 24 joints
Links:
- link base_link: mass 3.55209336 -> 3.23587253
- link left_ankle_pitch_link: mass 0.17366118 -> 0.16605731
- link left_ankle_roll_link: mass 0.78817642 -> 0.71237841
- link left_elbow_link: mass 0.81770364 -> 0.77922872
- link left_hip_pitch_link: mass 1.86216378 -> 1.83930168
- link left_hip_roll_link: mass 1.74387104 -> 1.45932598
- link left_hip_yaw_link: mass 2.57015343 -> 2.38381463
- link left_knee_link: mass 2.78730161 -> 2.45769202
- link left_shoulder_pitch_link: mass 0.83889911 -> 0.82850012
- link left_shoulder_roll_link: mass 0.80442734 -> 0.76916758
- link left_shoulder_yaw_link: mass 1.10463437 -> 0.95227320
- link left_wrist_roll_link: mass 0.15878030 -> 0.16115938
- link right_ankle_pitch_link: mass 0.17366118 -> 0.16605731
- link right_ankle_roll_link: mass 0.78817642 -> 0.71237841
- link right_elbow_link: mass 0.81744969 -> 0.77922499
- link right_hip_pitch_link: mass 1.86219733 -> 1.84174869
- link right_hip_roll_link: mass 1.74387104 -> 1.45932598
- link right_hip_yaw_link: mass 2.57008707 -> 2.38427565
- link right_knee_link: mass 2.78711852 -> 2.44960559
- link right_shoulder_pitch_link: mass 0.83890716 -> 0.82850796
- link right_shoulder_yaw_link: mass 1.08841996 -> 0.95225273
- link right_wrist_roll_link: mass 0.15878030 -> 0.16115938
- link waist_roll_link: mass 1.82887777 -> 1.53201882
- link waist_yaw_link: mass 8.02130808 -> 7.53658565
Joints:
- joint left_ankle_pitch_joint: origin xyz=0.03131 0.031811 -0.30533 rpy=0 0 0 -> xyz=0.03131 0.030811 -0.30533 rpy=0 0 0
- joint left_elbow_joint: origin xyz=0.020793 -0.031888 -0.10414 rpy=0 0 0 -> xyz=0.020796 -0.031888 -0.10414 rpy=0 0 0
- joint left_hip_pitch_joint: origin xyz=-0.03843 0.063987 -0.051639 rpy=0 0 0 -> xyz=-0.03843 0.062987 -0.051639 rpy=0 0 0
- joint left_hip_roll_joint: origin xyz=0.032915 0.060254 -0.060672 rpy=0 0 0 -> xyz=0.031915 0.061254 -0.060672 rpy=0 0 0
- joint left_hip_yaw_joint: origin xyz=-0.013698 0 -0.129 rpy=0 0 0 -> xyz=-0.012698 0 -0.129 rpy=0 0 0
- joint left_knee_joint: origin xyz=-0.033201 -0.031809 -0.16509 rpy=0 0 0 -> xyz=-0.033201 -0.030809 -0.16509 rpy=0 0 0
- joint left_shoulder_pitch_joint: origin xyz=0 0.1165 0.19949 rpy=0 0 0 -> xyz=0 0.116496194698121 0.19848715574272 rpy=0 0 0
- joint left_shoulder_roll_joint: origin xyz=0.028402 0.060357 -0.015009 rpy=0 0 0 -> xyz=0.0287432951006891 0.0653494445514435 -0.014608906526987 rpy=0 0 0
- joint left_shoulder_yaw_joint: origin xyz=-0.019058 0 -0.105 rpy=0 0 0 -> xyz=-0.0190574930004302 0 -0.105000039994097 rpy=0 0 0
- joint left_wrist_roll_joint: origin xyz=0.11609 0.031859 -0.018793 rpy=0 0 0 -> xyz=0.116093381994033 0.031859446289993 -0.0187927584979322 rpy=0 0 0
- joint right_ankle_pitch_joint: origin xyz=0.03131 -0.031809 -0.30533 rpy=0 0 0 -> xyz=0.03131 -0.030809 -0.30533 rpy=0 0 0
- joint right_elbow_joint: origin xyz=0.020793 0.031888 -0.10414 rpy=0 0 0 -> xyz=0.0207956801502895 0.031887525882762 -0.104135222723484 rpy=0 0 0
- joint right_hip_pitch_joint: origin xyz=-0.03843 -0.070013 -0.051639 rpy=0 0 0 -> xyz=-0.03843 -0.069013 -0.051639 rpy=0 0 0
- joint right_hip_roll_joint: origin xyz=0.032915 -0.060254 -0.060672 rpy=0 0 0 -> xyz=0.031915 -0.061254 -0.060672 rpy=0 0 0
- joint right_hip_yaw_joint: origin xyz=-0.013698 0 -0.129 rpy=0 0 0 -> xyz=-0.012698 0 -0.129 rpy=0 0 0
- joint right_knee_joint: origin xyz=-0.033201 0.031809 -0.16509 rpy=0 0 0 -> xyz=-0.0332010004232152 0.0308089665012395 -0.165090022909223 rpy=0 0 0
- joint right_shoulder_pitch_joint: origin xyz=0 -0.1165 0.19949 rpy=0 0 0 -> xyz=0 -0.116496194698064 0.198487155742749 rpy=0 0 0
- joint right_shoulder_roll_joint: origin xyz=0.028402 -0.060357 -0.015009 rpy=0 0 0 -> xyz=0.0287432951007422 -0.0653494445235536 -0.0146089065305009 rpy=0 0 0
- joint right_shoulder_yaw_joint: origin xyz=-0.019058 0 -0.105 rpy=0 0 0 -> xyz=-0.0190573923593691 0 -0.105000126276637 rpy=0 0 0
- joint right_wrist_roll_joint: origin xyz=0.11609 -0.031859 -0.018793 rpy=0 0 0 -> xyz=0.11609334409225 -0.031859369715491 -0.0187927299688337 rpy=0 0 0
- joint waist_roll_joint: origin xyz=-0.0065899 -0.0030127 0.052984 rpy=0 0 0 -> xyz=-0.00757994881845658 -0.00301269924435144 0.0529838303646947 rpy=0 0 0
- joint waist_yaw_joint: origin xyz=-0.031845 0 0.067 rpy=0 0 0 -> xyz=-0.0308449999997339 0 0.0679999999997294 rpy=0 0 0

Commit message: add head

File: urdf/rp1.urdf (robot description, URDF)
Before this commit: robot rp1.3.2, 29 links, 28 joints
Links:
- link waist_yaw_link: mass 7.53658565 -> 8.05985424

File: urdf/rp1_24dof.urdf (robot description, URDF)
Before this commit: robot rp1.3.2, 25 links, 24 joints
Links:
- link waist_yaw_link: mass 7.53658565 -> 8.05985424

Commit message: update ankle collision

File: urdf/rp1.urdf (robot description, URDF)
Before this commit: robot rp1.3.2, 29 links, 28 joints
Links:
- link left_ankle_roll_link: geometry collision cylinder length=0.06 radius=0.01; collision cylinder length=0.06 radius=0.01
- link right_ankle_roll_link: geometry collision cylinder length=0.06 radius=0.01; collision cylinder length=0.06 radius=0.01

File: urdf/rp1_24dof.urdf (robot description, URDF)
Before this commit: robot rp1.3.2, 25 links, 24 joints
Links:
- link left_ankle_roll_link: geometry collision cylinder length=0.06 radius=0.01; collision cylinder length=0.06 radius=0.01
- link right_ankle_roll_link: geometry collision cylinder length=0.06 radius=0.01; collision cylinder length=0.06 radius=0.01

Commit message: update mass

File: urdf/rp1.urdf (robot description, URDF)
Before this commit: robot rp1.3.2, 29 links, 28 joints
Links:
- link base_link: mass 3.23587253 -> 3.295
- link left_hip_roll_link: mass 1.45932598 -> 1.473
- link left_hip_yaw_link: mass 2.38381463 -> 2.483
- link left_knee_link: mass 2.45769202 -> 2.557
- link right_hip_roll_link: mass 1.45932598 -> 1.473
- link right_hip_yaw_link: mass 2.38427565 -> 2.483
- link right_knee_link: mass 2.44960559 -> 2.557
- link waist_yaw_link: mass 8.05985424 -> 7.8689

File: urdf/rp1_24dof.urdf (robot description, URDF)
Before this commit: robot rp1.3.2, 25 links, 24 joints
Links:
- link base_link: mass 3.23587253 -> 3.295
- link left_hip_roll_link: mass 1.45932598 -> 1.473
- link left_hip_yaw_link: mass 2.38381463 -> 2.483
- link left_knee_link: mass 2.45769202 -> 2.557
- link right_hip_roll_link: mass 1.45932598 -> 1.473
- link right_hip_yaw_link: mass 2.38427565 -> 2.483
- link right_knee_link: mass 2.44960559 -> 2.557
- link waist_yaw_link: mass 8.05985424 -> 7.8689

Commit message: update kkm version

File: urdf/rp1.urdf (robot description, URDF)
Before this commit: robot rp1.3.2, 29 links, 28 joints
Links:
- link left_ankle_roll_link: mass 0.71237841 -> 0.6430; geometry collision cylinder length=0.06 radius=0.01; collision cylinder length=0.06 radius=0.01
- link right_ankle_roll_link: mass 0.71237841 -> 0.6430; geometry collision cylinder length=0.06 radius=0.01; collision cylinder length=0.06 radius=0.01
- link waist_yaw_link: mass 7.8689 -> 8.3430

File: urdf/rp1_24dof.urdf (robot description, URDF)
Before this commit: robot rp1.3.2, 25 links, 24 joints
Links:
- link left_ankle_roll_link: mass 0.71237841 -> 0.6430; geometry collision cylinder length=0.06 radius=0.01; collision cylinder length=0.06 radius=0.01
- link right_ankle_roll_link: mass 0.71237841 -> 0.6430; geometry collision cylinder length=0.06 radius=0.01; collision cylinder length=0.06 radius=0.01
- link waist_yaw_link: mass 7.8689 -> 8.3430
