Commit message: update 24dof wrist

File: urdf/rp1_24dof.urdf (robot description, URDF)
Before this commit: robot rp1.3.2, 25 links, 24 joints
Links:
- removed link left_wrist_roll_link
- removed link right_wrist_roll_link
- added link left_wrist_link, mass 0.46025356; collision mesh filename=../meshes/left_wrist_link.STL; visual mesh filename=../meshes/left_wrist_link.STL
- added link right_wrist_link, mass 0.46029783; collision mesh filename=../meshes/right_wrist_link.STL; visual mesh filename=../meshes/right_wrist_link.STL
Joints:
- removed joint left_wrist_roll_joint
- removed joint right_wrist_roll_joint
- added joint left_wrist_joint: type revolute, parent left_elbow_link, child left_wrist_link, origin xyz=0.116093381994033 0.031859446289993 -0.0187927584979322 rpy=0 0 0, axis 1 0 0, limit lower=-2.56 upper=2.56 effort=35.3 velocity=21.88648
- added joint right_wrist_joint: type revolute, parent right_elbow_link, child right_wrist_link, origin xyz=0.11609334409225 -0.031859369715491 -0.0187927299688337 rpy=0 0 0, axis 1 0 0, limit lower=-2.56 upper=2.56 effort=35.3 velocity=21.88648
